Commit message: Criei um outro modelo urdf com as restrições de ângulos do pioneer, e o anterior renomei como piooner_7dof2

File: Simulacoes_Ros/pioneer_7dof2.urdf (robot description, URDF)
Before this commit: robot robotic_arm, 13 links, 12 joints
Joints:
- joint Five_joint: limit lower=-2.8798 upper=2.8798 effort=100.0 velocity=1.0 -> (none); type revolute -> continuous
- joint Four_joint: limit lower=-2.8798 upper=2.8798 effort=100.0 velocity=1.0 -> (none); type revolute -> continuous
- joint One_joint: limit lower=-2.8798 upper=2.8798 effort=100.0 velocity=1.0 -> (none); type revolute -> continuous
- joint Seven_joint: limit lower=-2.8798 upper=2.8798 effort=100.0 velocity=1.0 -> (none); type revolute -> continuous
- joint Six_joint: limit lower=-2.8798 upper=2.8798 effort=100.0 velocity=1.0 -> (none); type revolute -> continuous
- joint Three_joint: limit lower=-2.8798 upper=2.8798 effort=100.0 velocity=1.0 -> (none); type revolute -> continuous
- joint Two_joint: limit lower=-1.5708 upper=1.5708 effort=100.0 velocity=1.0 -> (none); type revolute -> continuous
