Commit message: Corrigir as dimensoes do pioneer em relação ao robo real

File: Simulacoes_Ros/pioneer_7dof.urdf (robot description, URDF)
Before this commit: robot robotic_arm, 13 links, 12 joints
Links:
- link Aux: geometry collision cylinder length=0.025 radius=0.025; visual cylinder length=0.025 radius=0.025
- link Five: geometry collision cylinder length=0.095 radius=0.025; visual cylinder length=0.095 radius=0.025
- link Four: geometry collision cylinder length=0.05 radius=0.025; visual cylinder length=0.05 radius=0.025
- link Gripper_Base: geometry collision cylinder length=0.05 radius=0.025; visual cylinder length=0.05 radius=0.025
- link L_F: geometry collision box size=0.01 0.01 0.03; visual box size=0.01 0.01 0.03
- link One: geometry collision cylinder length=0.05 radius=0.025; visual cylinder length=0.05 radius=0.025
- link R_F: geometry collision box size=0.01 0.01 0.03; visual box size=0.01 0.01 0.03
- link Seven: geometry collision cylinder length=0.05 radius=0.025; visual cylinder length=0.05 radius=0.025
- link Six: geometry collision cylinder length=0.05 radius=0.025; visual cylinder length=0.05 radius=0.025
- link Three: geometry collision cylinder length=0.1 radius=0.025; visual cylinder length=0.1 radius=0.025
- link Two: geometry collision cylinder length=0.05 radius=0.025; visual cylinder length=0.05 radius=0.025
- link base_link: geometry collision box size=0.1 0.1 0.05; visual box size=0.1 0.1 0.05
Joints:
- joint Aux_joint: origin xyz=0.0 0.15 0.0 rpy=0.0 0.0 0.0 -> xyz=0.0 0.05 0.0 rpy=0.0 0.0 0.0
- joint Five_joint: origin xyz=0.0 0.0 0.3 rpy=1.5708 0.0 0.0 -> xyz=0.0 0.0 0.145 rpy=1.5708 0.0 0.0
- joint Gripper_Base_joint: origin xyz=0.0 0 -0.2 rpy=0.0 3.1416 0.0  -> xyz=0.0 0 -0.075 rpy=0.0 3.1416 0.0 
- joint L_F_joint: limit lower=-0.02 upper=0.02 effort=100.0 velocity=1.0 -> lower=-0.01 upper=0.01 effort=100.0 velocity=1.0; origin xyz=0.0 0.03 0.0 -> xyz=0.0 0.015 0.0
- joint One_joint: origin xyz=0.0 0.0 0.3 rpy=1.5708 0.0 1.5708 -> xyz=0.0 0.0 0.125 rpy=1.5708 0.0 1.5708
- joint R_F_joint: limit lower=0.02 upper=-0.02 effort=100.0 velocity=1.0 -> lower=0.01 upper=-0.01 effort=100.0 velocity=1.0; origin xyz=0.0 -0.03 0.0 -> xyz=0.0 -0.015 0.0
- joint Seven_joint: origin xyz=0.0 0.05 0.0 rpy=1.5708  1.5708  0.0 -> xyz=0.0 0.025 0.0 rpy=1.5708  1.5708  0.0
- joint Three_joint: origin xyz=0.0 0.0 0.3 rpy=1.5708 0.0 0.0 -> xyz=0.0 0.0 0.15 rpy=1.5708 0.0 0.0

File: Simulacoes_Ros/pioneer_7dof2.urdf (robot description, URDF)
Before this commit: robot robotic_arm, 13 links, 12 joints
Links:
- link Aux: geometry collision cylinder length=0.025 radius=0.025; visual cylinder length=0.025 radius=0.025
- link Five: geometry collision cylinder length=0.095 radius=0.025; visual cylinder length=0.095 radius=0.025
- link Four: geometry collision cylinder length=0.05 radius=0.025; visual cylinder length=0.05 radius=0.025
- link Gripper_Base: geometry collision cylinder length=0.05 radius=0.025; visual cylinder length=0.05 radius=0.025
- link L_F: geometry collision box size=0.01 0.01 0.03; visual box size=0.01 0.01 0.03
- link One: geometry collision cylinder length=0.05 radius=0.025; visual cylinder length=0.05 radius=0.025
- link R_F: geometry collision box size=0.01 0.01 0.03; visual box size=0.01 0.01 0.03
- link Seven: geometry collision cylinder length=0.05 radius=0.025; visual cylinder length=0.05 radius=0.025
- link Six: geometry collision cylinder length=0.05 radius=0.025; visual cylinder length=0.05 radius=0.025
- link Three: geometry collision cylinder length=0.1 radius=0.025; visual cylinder length=0.1 radius=0.025
- link Two: geometry collision cylinder length=0.05 radius=0.025; visual cylinder length=0.05 radius=0.025
- link base_link: geometry collision box size=0.1 0.1 0.05; visual box size=0.1 0.1 0.05
Joints:
- joint Aux_joint: origin xyz=0.0 0.15 0.0 rpy=0.0 0.0 0.0 -> xyz=0.0 0.05 0.0 rpy=0.0 0.0 0.0
- joint Five_joint: origin xyz=0.0 0.0 0.3 rpy=1.5708 0.0 0.0 -> xyz=0.0 0.0 0.145 rpy=1.5708 0.0 0.0
- joint Gripper_Base_joint: origin xyz=0.0 0 -0.2 rpy=0.0 3.1416 0.0  -> xyz=0.0 0 -0.075 rpy=0.0 3.1416 0.0 
- joint L_F_joint: limit lower=-0.02 upper=0.02 effort=100.0 velocity=1.0 -> lower=-0.01 upper=0.01 effort=100.0 velocity=1.0; origin xyz=0.0 0.03 0.0 -> xyz=0.0 0.015 0.0
- joint One_joint: origin xyz=0.0 0.0 0.3 rpy=1.5708 0.0 1.5708 -> xyz=0.0 0.0 0.125 rpy=1.5708 0.0 1.5708
- joint R_F_joint: limit lower=0.02 upper=-0.02 effort=100.0 velocity=1.0 -> lower=0.01 upper=-0.01 effort=100.0 velocity=1.0; origin xyz=0.0 -0.03 0.0 -> xyz=0.0 -0.015 0.0
- joint Seven_joint: origin xyz=0.0 0.05 0.0 rpy=1.5708  1.5708  0.0 -> xyz=0.0 0.025 0.0 rpy=1.5708  1.5708  0.0
- joint Three_joint: origin xyz=0.0 0.0 0.3 rpy=1.5708 0.0 0.0 -> xyz=0.0 0.0 0.15 rpy=1.5708 0.0 0.0

Commit message: Corrigi os limites de juntas do modelo pioneer_7dof.urdf

File: Simulacoes_Ros/pioneer_7dof.urdf (robot description, URDF)
Before this commit: robot robotic_arm, 13 links, 12 joints
Joints:
- joint Five_joint: limit lower=-2.8798 upper=2.8798 effort=100.0 velocity=1.0 -> lower=-2.6179 upper=2.6179 effort=100.0 velocity=1.0
- joint Four_joint: limit lower=-2.8798 upper=2.8798 effort=100.0 velocity=1.0 -> lower=-1.6144 upper=1.6144 effort=100.0 velocity=1.0
- joint One_joint: limit lower=-2.8798 upper=2.8798 effort=100.0 velocity=1.0 -> lower=-2.6179 upper=2.6179 effort=100.0 velocity=1.0
- joint Seven_joint: limit lower=-2.8798 upper=2.8798 effort=100.0 velocity=1.0 -> lower=-1.7889 upper=1.7889 effort=100.0 velocity=1.0
- joint Six_joint: limit lower=-2.8798 upper=2.8798 effort=100.0 velocity=1.0 -> lower=-1.8413 upper=1.8413 effort=100.0 velocity=1.0
- joint Three_joint: limit lower=-2.8798 upper=2.8798 effort=100.0 velocity=1.0 -> lower=-2.6179 upper=2.6179 effort=100.0 velocity=1.0
- joint Two_joint: limit lower=-1.5708 upper=1.5708 effort=100.0 velocity=1.0 -> lower=-1.5358 upper=1.5358 effort=100.0 velocity=1.0
